Commit message: Model is opening in Rviz. Prismatic joint for nut is been defined.

File: throt_control_description/xacro/robot.xacro (robot description, xacro)
@@ -3,10 +3,10 @@
   <link name="base_link">
     <visual>
-      <origin xyz="0 0 0" rpy="0 0 0"/>
+      <origin xyz="0 0 0" rpy="${pi/2} 0 0"/>
       <geometry>
-        <mesh filename="package://throt_control_description/throttle_control.stl" scale="0.001 0.001 0.001"/>
+        <mesh filename="package://throt_control_description/meshes/throttle_control.stl" scale="0.001 0.001 0.001"/>
       </geometry>
       <material name="acrylic">
-        <color rgba="1 0.9 1 0.8"/>
+        <color rgba="1 0.9 1 1"/>
       </material>
     </visual>
@@ -14,7 +14,31 @@
       <origin xyz="0 0 0" rpy="0 0 0"/>
       <geometry>
-        <mesh filename="package://throt_control_description/throttle_control.stl" scale="0.001 0.001 0.001"/>
+        <mesh filename="package://throt_control_description/meshes/throttle_control.stl" scale="0.001 0.001 0.001"/>
       </geometry>
     </collision>
   </link>
+  <link name="nut_assem">
+    <visual>
+      <origin xyz="0 0 0" rpy="0 0 -${pi/2}"/>
+      <geometry>
+        <mesh filename="package://throt_control_description/meshes/nut_assem.stl" scale="0.001 0.001 0.001"/>
+      </geometry>
+      <material name="grey">
+        <color rgba="0.4 0.4 0.4 1"/>
+      </material>
+    </visual>
+    <collision>
+      <origin xyz="0 0 0" rpy="0 0 0"/>
+      <geometry>
+        <mesh filename="package://throt_control_description/meshes/nut_assem.stl" scale="0.001 0.001 0.001"/>
+      </geometry>
+    </collision>
+  </link>
+  <joint name="base_link_nut_assem" type="prismatic">
+    <origin xyz="0.14 -0.020 0.016" rpy="0 0 0"/>
+    <parent link="base_link"/>
+    <child link="nut_assem"/>
+    <axis xyz="0 1 0"/>
+    <limit lower="-0.1" upper="0.1" effort="10" velocity="0.01"/>
+  </joint>
 </robot>

Commit message: Modified feedback.py added gui to description.

File: throt_control_description/xacro/robot.xacro (robot description, xacro)
@@ -39,6 +39,6 @@
     <parent link="base_link"/>
     <child link="nut_assem"/>
-    <axis xyz="0 1 0"/>
-    <limit lower="-0.1" upper="0.1" effort="10" velocity="0.01"/>
+    <axis xyz="1 0 0"/>
+    <limit lower="0.0" upper="-0.04" effort="10" velocity="0.01"/>
   </joint>
 </robot>
